Commit message: gari and agv1 incorporated

File: src/myagv_description/urdf/agv.urdf (robot description, URDF)
Before this commit: robot agv, 7 links, 6 joints
Links:
- added link default_cam
Joints:
- added joint default_cam_joint: type fixed, parent base_link, child default_cam, origin xyz=0.0 0.0 0.3 rpy=0.0 0.0 0.0
